File: piportable v7.2/portablePi v84.sch (KiCad schematic (older format))
At the start: 74 parts, among them IC1 Raspberry_Pi_Zero_W_(v1.3), J1 AudioJack3, SW0 SW_Push, SW1 SW_Push, SW10 SW_Push, SW11 SW_Push, SW12 SW_Push, SW13 SW_Push, SW14 SW_Push, SW15 SW_Push, SW16 SW_Push, SW17 SW_Push, SW18 SW_Push, SW19 SW_Push, SW2 SW_Push, SW20 SW_Push, SW21 SW_Push, SW22 SW_Push, SW23 SW_Push, SW24 SW_Push, SW25 SW_Push, SW26 SW_Push, SW27 SW_Push, SW28 SW_Push, SW29 SW_Push, SW3 SW_Push, SW30 SW_Push, SW31 SW_Push, SW32 SW_Push, SW33 SW_Push, SW34 SW_Push, SW35 SW_Push, SW36 SW_Push, SW37 SW_Push, SW38 SW_Push, SW39 SW_Push, SW4 SW_Push, SW40 SW_Push, SW41 SW_Push, SW42 SW_Push, SW43 SW_Push, SW44 SW_Push, SW45 SW_Push, SW46 SW_Push, SW47 SW_Push, SW48 SW_Push, SW49 SW_Push, SW5 SW_Push, SW50 SW_Push, SW51 SW_Push, SW52 SW_Push, SW53 SW_Push, SW54 SW_Push, SW55 SW_Push, SW56 SW_Push, SW6 SW_Push, SW7 SW_Push, SW8 SW_Push, SW9 SW_Push, U1 ATmega328P-PU, Y1 Crystal

Commit message: the last versions
Parts:
- removed D1, D10, D2, D3, D4, D5, D6, D7, D8, D9: D, Diode_THT:D_T-1_P10.16mm_Horizontal, symbol Device:D
- added D1, D10, D2, D3, D4, D5, D6, D7, D8, D9: 1N4148, Diode_THT:D_T-1_P5.08mm_Horizontal, symbol Diode:1N4148
- added U2, U3: PCF8574, Package_DIP:DIP-16_W10.16mm_LongPads, symbol Interface_Expansion:PCF8574
Connections:
- net labels added: SDA, SDL
Other:
- moved on the sheet: J1
